File: HardWare/Placas/Olivia_control_v0.1/v0.1/v0.1.kicad_pcb (KiCad board)
At the start: 2 copper layers, 100 x 70 mm, 50 parts, among them J1 PROG, J10 Motor_B, J11 I2C, J12 DAC, J13 UART2, J15 TRIAC_220VAC, J17 In12V, J18 LED_RGB, J2 Input1, J3 Input2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

Commit message: pcb primer borrador
Parts:
- removed D3: ledPlcc6, LED_SMD:LED_RGB_PLCC-6
- removed J18: LED_RGB, Connector_Molex:Molex_SL_171971-0004_1x04_P2.54mm_Vertical
- removed R13, R14, R15: R, Resistor_SMD:R_0805_2012Metric_Pad1.20x1.40mm_HandSolder
- added J6: LED, Connector_Molex:Molex_SL_171971-0003_1x03_P2.54mm_Vertical, B.Cu at (177.1, 68.8)
- C10, C11, C8, C9, F1, J10, J11, J12, J13, J2, J3, J4, J5, J8, J9, R10, R7, R8, R9, U2, U3, U5, U6: moved to B.Cu
- moved PS1 131.5 mm to (174.8, 128.5), turned to 180 degrees
- moved J5 111.9 mm to (120.0, 72.7), turned to 90 degrees
- moved J4 111.5 mm to (120.0, 82.0), turned to 90 degrees
- moved J3 110.7 mm to (120.0, 91.4), turned to 90 degrees
- moved J2 110.1 mm to (120.0, 100.8), turned to 90 degrees
- moved R4 100.2 mm to (113.7, 72.7), turned to 0 degrees
- moved R3 100.0 mm to (113.7, 82.0)
- moved C4 99.5 mm to (115.7, 79.5), turned to 0 degrees
- moved C5 99.5 mm to (115.8, 70.1), turned to 0 degrees
- moved R2 99.1 mm to (113.7, 91.5), turned to 0 degrees
- moved C3 98.5 mm to (115.7, 88.9), turned to 0 degrees
- moved R1 98.4 mm to (113.8, 100.7), turned to 0 degrees
- moved C2 97.7 mm to (115.6, 98.2), turned to 0 degrees
- moved J8 94.0 mm to (192.0, 51.9), turned to 180 degrees
- moved J12 85.5 mm to (129.8, 57.9), turned to -90 degrees
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Connections:
- net /TX2 renamed /D_led
Routing:
- net GND: track 0.00 -> 695.5 mm, vias 0 -> 4
- net +3.3V: track 0.00 -> 271.2 mm, vias 0 -> 5
- net +3.3V_fused: track 0.00 -> 133.5 mm, vias 0 -> 3
- net /FASE: track 0.00 -> 125.1 mm
- net /EN: track 0.00 -> 106.4 mm, vias 0 -> 1
- net /NEUTRO: track 0.00 -> 103.0 mm
- net /In1: track 0.00 -> 81.4 mm
- net /In2: track 0.00 -> 70.6 mm
- net /EN_B: track 0.00 -> 62.0 mm, vias 0 -> 2
- net /TXD0: track 0.00 -> 59.2 mm, vias 0 -> 1
- net /ZERO: track 0.00 -> 59.2 mm, vias 0 -> 1
- net /TRIAC_A: track 0.00 -> 59.1 mm, vias 0 -> 1
- net /In3: track 0.00 -> 58.0 mm
- net /RXD0: track 0.00 -> 53.0 mm, vias 0 -> 1
- net Net-(PS1-+Vout): track 0.00 -> 49.9 mm
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- added copper zone on B.Cu, net +3.3V
- added copper zone on B.Cu, net GND
- added copper zone on F.Cu, net GND
Other:
- board size 100 x 70 mm -> 100 x 100 mm
