File: HardWare/Placas/Olivia_control_v0.1/v0.1/v0.1.kicad_sch (KiCad schematic)
At the start: 50 parts, among them J1 PROG, J10 Motor_B, J11 I2C, J12 DAC, J13 UART2, J15 TRIAC_220VAC, J17 In12V, J18 LED_RGB, J2 Input1, J3 Input2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

Commit message: pcb primer borrador
Parts:
- removed D3: ledPlcc6, LED_SMD:LED_RGB_PLCC-6, symbol LED:CLX6F-FKC
- removed J18: LED_RGB, Connector_Molex:Molex_SL_171971-0004_1x04_P2.54mm_Vertical, symbol Connector_Generic:Conn_01x04
- removed R13, R14, R15: R, Resistor_SMD:R_0805_2012Metric_Pad1.20x1.40mm_HandSolder, symbol Device:R
- added J6: LED, Connector_Molex:Molex_SL_171971-0003_1x03_P2.54mm_Vertical, symbol Connector_Generic:Conn_01x03
Connections:
- net +3.3V_fused: now also J6.3 (Pin_3)
- net GND: now also J6.1 (Pin_1)
- net TX2 renamed D_led
- net D_led: now also J6.2 (Pin_2)
Other:
- moved on the sheet: J10, J12, J9
